File: Main.kicad_pcb (KiCad board)
At the start: 2 copper layers, 0 parts

Commit message: More final schematic, module footprints
Added all the footprints we need to a library, made a link file from
part schematics to footprints, everything's ready to be laid out/routed
Parts:
- added C1: 18pF, SM0402_c, F.Cu at (0.00, 0.00)
- added C10, C12, C14, C16, C17, C18, C19, C22, C23, C24, C25, C26, C27, C28, C29, C30, C31, C33, C34, C35, C38, C40, C5, C52: 100nF, SM0402_c, F.Cu at (0.00, 0.00)
- added C11, C39, C47: 10uF, SM0603_Capa, F.Cu at (0.00, 0.00)
- added C13, C15, C2: 22pF, SM0402_c, F.Cu at (0.00, 0.00)
- added C20, C36: 1uF, SM0402_c, F.Cu at (0.00, 0.00)
- added C21: 47pF, SM0402_c, F.Cu at (0.00, 0.00)
- added C3, C37, C41: 2.2uF, SM0402_c, F.Cu at (0.00, 0.00)
- added C32: 4n7, SM0402_c, F.Cu at (0.00, 0.00)
- added C4, C44: 4.7uF, SM0603_Capa, F.Cu at (0.00, 0.00)
- added C42: 10nF, SM0402_c, F.Cu at (0.00, 0.00)
- added C43, C45, C46, C48, C49, C50: .1uF, SM0402_c, F.Cu at (0.00, 0.00)
- added C51: C, SM0603_Capa, F.Cu at (0.00, 0.00)
- added C6, C7, C8, C9: C, SM0402_c, F.Cu at (0.00, 0.00)
- added CON1: USB-MINI-B, MICRO-B_USB, F.Cu at (0.00, 0.00)
- added D1, D2: LED, LED-0603, F.Cu at (0.00, 0.00)
- added L1, L2: INDUCTOR, SM0402, F.Cu at (0.00, 0.00)
- added L3: 10uH, SM1210, F.Cu at (0.00, 0.00)
- added P1: CONN_6, SIL-6, F.Cu at (0.00, 0.00)
- added R1, R10, R11, R12, R13, R14, R2, R3, R5, R6, R7: 10K, SM0402_r, F.Cu at (0.00, 0.00)
- added R15: 2K, SM0402_r, F.Cu at (0.00, 0.00)
- added R4: 1M, SM0402_r, F.Cu at (0.00, 0.00)
- added R8, R9: 68, SM0402_r, F.Cu at (0.00, 0.00)
- added SW1, SW2: TACT, TACT_SWITCH, F.Cu at (0.00, 0.00)
- added U1: AS4C8M16S, TSOP2_54, F.Cu at (0.00, 0.00)
- added U10: N25Q128A, psop-8, F.Cu at (0.00, 0.00)
- added U11: FPC_50, FPC ZIF 50, F.Cu at (0.00, 0.00)
- added U2: M10478, GPS_M10478, F.Cu at (0.00, 0.00)
- added U3: LM3670, SOT23-5, F.Cu at (0.00, 0.00)
- added U4: XBEE, XBEE, F.Cu at (0.00, 0.00)
- added U5: STM32F429_144, LQFP144, F.Cu at (0.00, 0.00)
- added U6: MPL3115A2, LGA_8, F.Cu at (0.00, 0.00)
- added U7: MPU-9250, QFN24_.4, F.Cu at (0.00, 0.00)
- added U8: RT9169, SOT23, F.Cu at (0.00, 0.00)
- added U9: MCP7383X, sot323-5, F.Cu at (0.00, 0.00)
- added X1: 32.768MHz, CRYSTAL_CPFB_SMD, F.Cu at (0.00, 0.00)
- added X2: 8MHz, CRYSTAL_CPFB_SMD, F.Cu at (0.00, 0.00)

Commit message: Board halfway routed, yay
Parts:
- removed C10: 100nF, SM0402_c
- added P2: CONN_2, SIL-2, F.Cu at (166.0, 116.2)
- C51: value C -> 4.7uF
- moved L1 281.3 mm to (229.3, 162.9), turned to 180 degrees
- moved C5 281.1 mm to (234.5, 155.0), turned to 90 degrees
- moved C4 280.8 mm to (232.0, 158.2)
- moved C1 280.3 mm to (228.9, 161.7), turned to 90 degrees
- moved L2 279.8 mm to (229.3, 160.3), turned to 180 degrees
- moved U3 279.2 mm to (232.2, 155.0)
- moved C3 278.8 mm to (229.5, 158.2)
- moved C2 278.1 mm to (229.5, 157.0)
- moved L3 277.3 mm to (232.2, 151.5)
- moved C11 276.8 mm to (229.5, 154.8), turned to 90 degrees
- moved U2 274.6 mm to (223.0, 160.2), turned to 180 degrees
- moved C16 274.4 mm to (237.5, 137.5), turned to 270 degrees
- moved C14 271.5 mm to (237.5, 131.5), turned to 90 degrees
- moved R1 270.6 mm to (224.8, 150.8), turned to 90 degrees
- moved C24 270.2 mm to (216.5, 161.6)
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Connections:
- C32 pad 1: N-0000017 -> N-0000088
- C51 pad 1: (no net) -> +5V
- L3 pad 1: (no net) -> N-0000066
- R4 pad 1: N-0000017 -> N-0000088
- U3 pad 4: (no net) -> +1.8V
- U3 pad 5: (no net) -> N-0000066
- U5 pad 1: /SW1 -> /LED1
- U5 pad 2: /SW2 -> /LED2
- U5 pad 3: /LED1 -> /SW1
- U5 pad 4: /LED2 -> /SW2
Routing:
- net /NRST: track 0.00 -> 73.5 mm, vias 0 -> 2
- net /BAT_SENSE: track 0.00 -> 57.3 mm, vias 0 -> 2
- net /BAT_DRIVE: track 0.00 -> 57.1 mm, vias 0 -> 2
- net /B7: track 0.00 -> 56.6 mm, vias 0 -> 2
- net /B6: track 0.00 -> 55.7 mm, vias 0 -> 2
- net /SDCLK: track 0.00 -> 51.1 mm, vias 0 -> 2
- net /A10: track 0.00 -> 50.9 mm, vias 0 -> 4
- net /NBL1: track 0.00 -> 48.8 mm, vias 0 -> 2
- net /B5: track 0.00 -> 48.7 mm, vias 0 -> 4
- net /SDCKE1: track 0.00 -> 47.2 mm, vias 0 -> 2
- net /CSX: track 0.00 -> 45.3 mm, vias 0 -> 4
- net /G2: track 0.00 -> 41.6 mm, vias 0 -> 4
- net /SWO: track 0.00 -> 41.4 mm, vias 0 -> 3
- net /G4: track 0.00 -> 41.2 mm, vias 0 -> 2
- net /A4: track 0.00 -> 41.1 mm, vias 0 -> 4
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Other:
- board outline added: 74.2 x 58 mm
- net class Default: clearance 0.254 -> 0.1524; trace_width 0.254 -> 0.1524; via_dia 0.889 -> 0.6858; via_drill 0.635 -> 0.3302
- rule trace_clearance: 0.254 -> 0.1524
- rule trace_min: 0.254 -> 0.1524
- rule via_min_drill: 0.508 -> 0.3302
- rule via_min_size: 0.889 -> 0.6858
