File: Main.kicad_pcb (KiCad board)
At the start: 2 copper layers, 74.2 x 58 mm, 88 parts, among them CON1 USB-MINI-B, P1 CONN_6, P2 CONN_2, SW1 TACT, SW2 TACT, U1 AS4C8M16S, U10 N25Q128A, U11 FPC_50, U2 M10478, U3 LM3670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

Commit message: Final ish board
Parts:
- renumbered P2 to BATTERY, D1 to LED1, D2 to LED2
Routing:
- net VDD: track 220.9 -> 236.3 mm, vias 26 -> 27
- net (no net): track 0.58 -> 6.72 mm, vias 0 -> 2
Other:
- board text added: "+"
- board text added: "-"
- board text added: "Banks Hunter 2.009 Pink Team Proxband 10/2014"
- board text added: "GND"
- board text added: "VDD"
