File: Main.sch (KiCad schematic (older format))
At the start: 1 part

Commit message: Initial micro data buses in place
Parts:
- added C? (x6): C, ~, symbol C
- added C? (x2): 2.2uF, ~, symbol C
- added R?: R, ~, symbol R
- added U?: RT9169, ~, symbol RT9169
- added U?: MCP7383X, MODULE, symbol MCP7383X
- added U?: MPL3115A2, MODULE, symbol MPL3115A2
- added X?: 32.768MHz, ~, symbol CRYSTAL
- added X?: 8MHz, ~, symbol CRYSTAL
Connections:
- net labels added: +BATT, A0, A1, A10, A11, A2, A3, A4, A5, A6, A7, A8, A9, B2, B3, B4, B5, B6, B7, BARO_SCL, BARO_SDA, CHARGE_STAT, D0, D1, D10, D11, D12, D13, D14, D15, D2, D3, D4, D5, D6, D7, D8, D9, G2, G3, G4, G5, G6, G7, GND, HSYNC, LCD_CLK, OSC32_IN, OSC32_OUT, OSC_IN, OSC_OUT, R2, R3, R4, R5, R6, R7, SDRAM_CLK, SDRAM_NWE, SDRAM_~CAS, VDD, VSYNC
- wire segments 0 -> 121

Commit message: Schematic done-ish
Parts:
- added C1: 18pF, ~, symbol C
- added C10: C, ~, symbol C
- added C11, C13, C15, C17, C18, C19, C20, C23, C24, C25, C26, C27, C28, C29, C30, C31, C32, C33, C34, C35, C38, C40, C50: 100nF, ~, symbol C
- added C12, C39, C46: 10uF, ~, symbol C
- added C14, C16, C2, C5: 22pF, ~, symbol C
- added C21, C36: 1uF, ~, symbol C
- added C22: 47pF, ~, symbol C
- added C3: 2.2uF, ~, symbol C
- added C4: 4.7uF, ~, symbol C
- added C42: 10nF, ~, symbol C
- added C43, C44, C47, C49: .1uF, ~, symbol C
- added D1, D2: LED, ~, symbol LED
- added L1, L2, L3: INDUCTOR, ~, symbol INDUCTOR
- added P1: CONN_6, symbol CONN_6
- added R1, R11, R12, R13, R14, R15, R2, R5, R6, R7, R8: 10K, ~, symbol R
- added R10, R9: 68, ~, symbol R
- added R3: 100K, ~, symbol R
- added R4: 200L, ~, symbol R
- added SW1, SW2: TACT, ~, symbol TACT
- added U1: AS4C8M16S, ~, symbol AS4C8M16S
- added U10: N25Q128A, symbol N25Q128A
- added U11: FPC_50, symbol FPC_50
- added U2: M10478, symbol M10478
- added U3: FT440, symbol FT440
- added U4: XBEE, ~, symbol XBEE
- added U7: MPU-9250, MODULE, symbol MPU-9250
- C45, C48: renamed from C?; value C -> .1uF
- R16: renamed from R?; value R -> 2K
- gave numbers to parts that had none: 12
Connections:
- net labels added: +1.8V, ANT_IN, ANT_OUT, BA0, BA1, BARO_INT, BAT_DRIVE, BAT_SENSE, BUCK_EN, CSX, DCX_SCL, DOTCLK, FL_CS, FL_HOLD, FL_MISO, FL_MOSI, FL_SCK, FL_WP, GPS_CTS, GPS_ONOFF, GPS_RX, GPS_TX, GPS_WAKEUP, IM0, IM1, IM2, IM3, IMU_INT, IMU_SCL, IMU_SDA, LCD_EN, LCD_RST, LCD_SDA, LED1, LED2, NBL0, NBL1, NRST, RDX, SDCKE1, SDCLK, SDNCAS, SDNE1, SDNRAS, SDNWE, SW1, SW2, SWCLK, SWDIO, SWO, TE, WRX_DCX, X+, X-, XB_DIN, XB_DOUT, XB_RST, Y+, Y-
- net labels removed: LCD_CLK, SDRAM_CLK, SDRAM_NWE, SDRAM_~CAS
- wire segments 121 -> 404
- no-connect marks 0 -> 55
Other:
- note added: "Micro bus caps"
- note added: "SDRAM bus caps"
- moved on the sheet: C37, C41, C45, C48, C6, C7, C8, C9, R16, U5, U6, U8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

Commit message: Added footprints of barometer and FPC-50
Also added USB to schematic
Parts:
- added C?: 4.7uF, ~, symbol C
- added C?: C, ~, symbol C
- added C?: 4n7, ~, symbol C
- added CON?: USB-MINI-B, symbol USB-MINI-B
- added R?: 1M, ~, symbol R
Connections:
- net labels added: +5V, USB_DM, USB_DP
- wire segments 404 -> 418
- no-connect marks 55 -> 54
Other:
- moved on the sheet: C38, C39, C40, U6

Commit message: Redid schematic annotation
Parts:
- gave numbers to parts that had none: 5
- renumbered C33 to C34, C34 to C35, C35 to C36, C36 to C37, C37 to C38, C38 to C39, C39 to C40, C40 to C41, C41 to C42, C42 to C43, C43 to C44, C44 to C46, C45 to C47, C46 to C48, C47 to C49, C48 to C50, C49 to C51, C50 to C53, R9 to R10, R10 to R11, R11 to R12, R12 to R13, R13 to R14, R14 to R15, R15 to R16, R16 to R17, R6 to R7, R7 to R8, R8 to R9

Commit message: More final schematic, module footprints
Added all the footprints we need to a library, made a link file from
part schematics to footprints, everything's ready to be laid out/routed
Parts:
- removed C10: C, ~, symbol C
- removed R3: 100K, ~, symbol R
- removed R4: 200L, ~, symbol R
- removed U3: FT440, symbol FT440
- added U3: LM3670, ~, symbol LM3670
- C5: value 22pF -> 100nF
- C51: renamed from C52; value C -> 4.7uF
- L3: value INDUCTOR -> 10uH
- renumbered C11 to C10, C12 to C11, C13 to C12, C14 to C13, C15 to C14, C16 to C15, C17 to C16, C18 to C17, C19 to C18, C20 to C19, C21 to C20, C22 to C21, C23 to C22, C24 to C23, C25 to C24, C26 to C25, C27 to C26, C28 to C27, C29 to C28, C30 to C29, C31 to C30, C32 to C31, C33 to C32, C34 to C33, C35 to C34, C36 to C35, C37 to C36, C38 to C37, C39 to C38, C40 to C39, C41 to C40, C42 to C41, C43 to C42, C44 to C43, C45 to C44, C46 to C45, C47 to C46, C48 to C47, C49 to C48, C50 to C49, C51 to C50, C53 to C52, R12 to R10, R13 to R11, R14 to R12, R15 to R13, R16 to R14, R17 to R15, R5 to R3, R6 to R4, R7 to R5, R8 to R6, R9 to R7, R10 to R8, R11 to R9
Connections:
- wire segments 418 -> 419
- no-connect marks 54 -> 53

Commit message: Board halfway routed, yay
Parts:
- removed C10: 100nF, ~, symbol C
- added P2: CONN_2, symbol CONN_2
Connections:
- wire segments 419 -> 429
- no-connect marks 53 -> 54

Commit message: Finished routing
Parts:
- removed C9: C, ~, symbol C
- removed X2: 8MHz, ~, symbol CRYSTAL
- added X2: 8MHz, ~, symbol CRYSTAL4
- C6, C7: value C -> 12.5pF
- C8: value C -> 10nF
Connections:
- net labels added: OSC_EN
- wire segments 429 -> 435
Changed lines of the file:
@@
 P 3050 7650
 F 0 "C6" H 3050 7750 40  0000 L CNN
-F 1 "C" H 3056 7565 40  0000 L CNN
+F 1 "12.5pF" H 3056 7565 40  0000 L CNN
 F 2 "~" H 3088 7500 30  0000 C CNN
 F 3 "~" H 3050 7650 60  0000 C CNN
@@
 P 3050 8250
 F 0 "C7" H 3050 8350 40  0000 L CNN
-F 1 "C" H 3056 8165 40  0000 L CNN
+F 1 "12.5pF" H 3056 8165 40  0000 L CNN
 F 2 "~" H 3088 8100 30  0000 C CNN
 F 3 "~" H 3050 8250 60  0000 C CNN
@@
 OSC32_OUT
 $Comp
-L CRYSTAL X2
-U 1 1 544FDEAF
-P 3250 9800
-F 0 "X2" H 3250 9950 60  0000 C CNN
-F 1 "8MHz" H 3250 9650 60  0000 C CNN
-F 2 "~" H 3250 9800 60  0000 C CNN
-F 3 "~" H 3250 9800 60  0000 C CNN
-	1    3250 9800
-	0    1    1    0
-$EndComp
-$Comp
-L C C8
-U 1 1 544FDEB5
-P 3050 9500
-F 0 "C8" H 3050 9600 40  0000 L CNN
-F 1 "C" H 3056 9415 40  0000 L CNN
-F 2 "~" H 3088 9350 30  0000 C CNN
-F 3 "~" H 3050 9500 60  0000 C CNN
-	1    3050 9500
-	0    1    1    0
-$EndComp
-$Comp
-L C C9
-U 1 1 544FDEBB
-P 3050 10100
-F 0 "C9" H 3050 10200 40  0000 L CNN
-F 1 "C" H 3056 10015 40  0000 L CNN
-F 2 "~" H 3088 9950 30  0000 C CNN
-F 3 "~" H 3050 10100 60  0000 C CNN
-	1    3050 10100
-	0    1    1    0
-$EndComp
-$Comp
 L GND #PWR026
 U 1 1 544FDEC2
-P 2850 10300
-F 0 "#PWR026" H 2850 10300 30  0001 C CNN
-F 1 "GND" H 2850 10230 30  0001 C CNN
-F 2 "" H 2850 10300 60  0000 C CNN
-F 3 "" H 2850 10300 60  0000 C CNN
-	1    2850 10300
+P 3050 9800
+F 0 "#PWR026" H 3050 9800 30  0001 C CNN
+F 1 "GND" H 3050 9730 30  0001 C CNN
+F 2 "" H 3050 9800 60  0000 C CNN
+F 3 "" H 3050 9800 60  0000 C CNN
+	1    3050 9800
 	1    0    0    -1
 $EndComp
-Text Label 3350 9500 0    60   ~ 0
+Text Label 4500 9700 0    60   ~ 0
 OSC_IN
-Text Label 3350 10100 0    60   ~ 0
+Text Label 4700 10350 0    60   ~ 0
 OSC_OUT
 $Comp
@@
 	1    0    0    -1
 $EndComp
-Text Label 5850 10550 0    60   ~ 0
+Text Label 5850 7150 0    60   ~ 0
 GPS_WAKEUP
 $Comp
@@
 	1    0    0    -1
 $EndComp
-Text Label 5850 9850 0    60   ~ 0
+Text Label 5850 7050 0    60   ~ 0
 GPS_ONOFF
-Text Label 8150 12000 1    60   ~ 0
+Text Label 6300 7450 2    60   ~ 0
 BUCK_EN
 Text Label 12100 10550 0    60   ~ 0
@@
 Text Label 6050 7350 0    60   ~ 0
 SW2
-Text Label 6050 7050 0    60   ~ 0
+Text Label 6050 9850 0    60   ~ 0
 LED1
-Text Label 6050 7150 0    60   ~ 0
+Text Label 6050 10550 0    60   ~ 0
 LED2
 Text Label 5850 9250 0    60   ~ 0
@@
 Text Label 5850 9350 0    60   ~ 0
 OSC_OUT
-NoConn ~ 6400 9650
 NoConn ~ 6400 7650
-NoConn ~ 6400 7450
 NoConn ~ 8150 6000
 NoConn ~ 8950 6000
@@
 	3250 8250 3750 8250
 Wire Wire Line
-	2850 9500 2850 10300
-Connection ~ 2850 10100
-Wire Wire Line
-	3250 9500 3750 9500
+	4400 9700 4900 9700
 Wire Wire Line
-	3250 10100 3750 10100
+	4600 10350 5100 10350
 Wire Wire Line
 	17850 3300 18150 3300
@@
 	6400 10450 5850 10450
 Wire Wire Line
-	6400 10550 5850 10550
+	6400 7150 5850 7150
 Wire Wire Line
 	7850 11600 7850 11950
@@
 Connection ~ 5250 950
 Wire Wire Line
-	6400 9850 5850 9850
-Wire Wire Line
-	8150 11600 8150 12000
+	6400 7050 5850 7050
 Wire Wire Line
 	12000 10550 12500 10550
@@
 	6400 7350 6050 7350
 Wire Wire Line
-	6400 7050 6050 7050
+	6400 9850 6050 9850
 Wire Wire Line
-	6400 7150 6050 7150
+	6400 10550 6050 10550
 Wire Wire Line
 	6400 9250 5850 9250
@@
 Connection ~ 3250 7650
 Connection ~ 3250 8250
-Connection ~ 3250 9500
-Connection ~ 3250 10100
+Connection ~ 4400 9700
+Connection ~ 4600 10350
 Wire Wire Line
 	5250 1350 5250 1400
@@
 Wire Wire Line
 	16750 3900 16850 3900
+$Comp
+L CRYSTAL4 X2
+U 1 1 5450E187
+P 4100 9800
+F 0 "X2" H 4100 9950 60  0000 C CNN
+F 1 "8MHz" H 4100 9650 60  0000 C CNN
+F 2 "~" H 4100 9800 60  0000 C CNN
+F 3 "~" H 4100 9800 60  0000 C CNN
+	1    4100 9800
+	1    0    0    -1
+$EndComp
+$Comp
+L C C8
+U 1 1 5450E1B0
+P 3350 9700
+F 0 "C8" H 3350 9800 40  0000 L CNN
+F 1 "10nF" H 3356 9615 40  0000 L CNN
+F 2 "~" H 3388 9550 30  0000 C CNN
+F 3 "~" H 3350 9700 60  0000 C CNN
+	1    3350 9700
+	0    -1   -1   0
+$EndComp
+Wire Wire Line
+	3550 9700 3800 9700
+$Comp
+L VDD #PWR0110
+U 1 1 5450E481
+P 3550 9700
+F 0 "#PWR0110" H 3550 9800 30  0001 C CNN
+F 1 "VDD" H 3550 9810 30  0000 C CNN
+F 2 "" H 3550 9700 60  0000 C CNN
+F 3 "" H 3550 9700 60  0000 C CNN
+	1    3550 9700
+	1    0    0    -1
+$EndComp
+Connection ~ 3550 9700
+$Comp
+L GND #PWR0111
+U 1 1 5450E9AB
+P 4450 10000
+F 0 "#PWR0111" H 4450 10000 30  0001 C CNN
+F 1 "GND" H 4450 9930 30  0001 C CNN
+F 2 "" H 4450 10000 60  0000 C CNN
+F 3 "" H 4450 10000 60  0000 C CNN
+	1    4450 10000
+	1    0    0    -1
+$EndComp
+Wire Wire Line
+	4450 10000 4450 9900
+Wire Wire Line
+	4450 9900 4400 9900
+Wire Wire Line
+	3050 9800 3050 9700
+Wire Wire Line
+	3050 9700 3150 9700
+Wire Wire Line
+	3300 9900 3800 9900
+Text Label 3300 9900 0    60   ~ 0
+OSC_EN
+NoConn ~ 4600 10350
+Wire Wire Line
+	6400 9650 5850 9650
+Text Label 5850 9650 0    60   ~ 0
+OSC_EN
+NoConn ~ 8150 11600
+Wire Wire Line
+	6400 7450 5900 7450
 $EndSCHEMATC
