File: rf/rf.sch (KiCad schematic (older format))
At the start: 45 parts, among them P1 CONN_1, P2 CONN_7, U1 SE2435L, U2 ADF7023, X1 CRYSTAL

Commit message: fixed net list and BOM
Parts:
- C1, C2, C3: footprint 0402 -> SM0402_c
- C12: footprint SM0402_c -> SM0603_Capa
- C23, C24: value 220nF -> 9pF
- C4: footprint 0603 -> SM0603_Capa
- C5: footprint 0201 -> SM0402_c
- P1: footprint (none) -> SIL-1
- P2: footprint (none) -> SIL-7
- X1: Frequency (none) -> 26MHz
Other:
- note added: "Capacitor should be split into 2?"
- note added: "Could be 0402"
- note added: "Make sure to drill hole for tension relief"
- note added: "Reconfigure GPIO pins. For example,\natb4 can be set for LNA enable"
- note added: "Should be 0603"
Changed lines of the file:
@@
 Sheet 1 1
 Title ""
-Date "11 nov 2014"
+Date "20 nov 2014"
 Rev ""
 Comp ""
@@
 P 8600 5600
 F 0 "C23" H 8600 5700 40  0000 L CNN
-F 1 "220nF" H 8606 5515 40  0000 L CNN
+F 1 "9pF" H 8606 5515 40  0000 L CNN
 F 2 "SM0402_c" H 8638 5450 30  0001 C CNN
 F 3 "~" H 8600 5600 60  0000 C CNN
@@
 P 9200 5600
 F 0 "C24" H 9200 5700 40  0000 L CNN
-F 1 "220nF" H 9206 5515 40  0000 L CNN
+F 1 "9pF" H 9206 5515 40  0000 L CNN
 F 2 "SM0402_c" H 9238 5450 30  0001 C CNN
 F 3 "~" H 9200 5600 60  0000 C CNN
@@
 F 2 "crystal_FA238-TSX3225" H 8900 5250 60  0001 C CNN
 F 3 "~" H 8900 5250 60  0000 C CNN
+F 4 "26MHz" H 8900 5250 60  0001 C CNN "Frequency"
 	1    8900 5250
 	1    0    0    -1
@@
 F 0 "C1" H 1450 3250 40  0000 L CNN
 F 1 "3.3pF" H 1456 3065 40  0000 L CNN
-F 2 "0402" H 1488 3000 30  0001 C CNN
+F 2 "SM0402_c" H 1488 3000 30  0001 C CNN
 F 3 "~" H 1450 3150 60  0000 C CNN
 	1    1450 3150
@@
 F 0 "C2" H 1500 3800 40  0000 L CNN
 F 1 "3.3pF" H 1506 3615 40  0000 L CNN
-F 2 "0402" H 1538 3550 30  0001 C CNN
+F 2 "SM0402_c" H 1538 3550 30  0001 C CNN
 F 3 "~" H 1500 3700 60  0000 C CNN
 	1    1500 3700
@@
 F 0 "C3" H 1500 4700 40  0000 L CNN
 F 1 "10pF" H 1506 4515 40  0000 L CNN
-F 2 "0402" H 1538 4450 30  0001 C CNN
+F 2 "SM0402_c" H 1538 4450 30  0001 C CNN
 F 3 "~" H 1500 4600 60  0000 C CNN
 	1    1500 4600
@@
 F 0 "C5" H 3150 5950 40  0000 L CNN
 F 1 "1nF" H 3156 5765 40  0000 L CNN
-F 2 "0201" H 3188 5700 30  0001 C CNN
+F 2 "SM0402_c" H 3188 5700 30  0001 C CNN
 F 3 "~" H 3150 5850 60  0000 C CNN
 	1    3150 5850
@@
 F 0 "C4" H 2700 5950 40  0000 L CNN
 F 1 "4.7uF" H 2706 5765 40  0000 L CNN
-F 2 "0603" H 2738 5700 30  0001 C CNN
+F 2 "SM0603_Capa" H 2738 5700 30  0001 C CNN
 F 3 "~" H 2700 5850 60  0000 C CNN
 	1    2700 5850
@@
 F 0 "C12" H 6300 4400 40  0000 L CNN
 F 1 "10uF" H 6306 4215 40  0000 L CNN
-F 2 "SM0402_c" H 6338 4150 30  0001 C CNN
+F 2 "SM0603_Capa" H 6338 4150 30  0001 C CNN
 F 3 "~" H 6300 4300 60  0000 C CNN
 	1    6300 4300
@@
 F 0 "P2" V 10920 2900 60  0000 C CNN
 F 1 "CONN_7" V 11020 2900 60  0000 C CNN
-F 2 "" H 10950 2900 60  0001 C CNN
+F 2 "SIL-7" H 10950 2900 60  0001 C CNN
 F 3 "" H 10950 2900 60  0000 C CNN
 	1    10950 2900
@@
 F 0 "P1" H 680 2800 40  0000 L CNN
 F 1 "CONN_1" H 600 2855 30  0001 C CNN
-F 2 "" H 600 2800 60  0001 C CNN
+F 2 "SIL-1" H 600 2800 60  0001 C CNN
 F 3 "" H 600 2800 60  0000 C CNN
 	1    600  2800
@@
 Wire Wire Line
 	7300 1750 7300 1800
+Text Notes 6950 3300 0    60   ~ 0
+Could be 0402
+Text Notes 2400 5900 0    60   ~ 0
+Should be 0603
+Text Notes 5950 4350 0    60   ~ 0
+Should be 0603
+Text Notes 750  4600 0    60   ~ 0
+Capacitor should be split into 2?
+Text Notes 300  2800 0    60   ~ 0
+Make sure to drill hole for tension relief
+Text Notes 9100 4000 0    60   ~ 0
+Reconfigure GPIO pins.  For example,\natb4 can be set for LNA enable
 $EndSCHEMATC
